File: server_lader.kicad_pcb (KiCad board)
At the start: 2 copper layers, 56 parts, among them IC1 ATMEGA168PA-A, IC2 DAC8560, P1 5V_Vbatt, P11 on/off, P12 A_regulation_out, P3 CONN_02X03, P4 I2C, P7 UART, P9 Drehrad, U2 LTV-356T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

Commit message: work
Parts:
- added C24: 1uF, SMD_Packages:SMD-0603, F.Cu at (175.3, 114.3)
- added D1: ZENER 5,6V, Diodes_SMD:Diode-Universal-SMA-SMB_Handsoldering, F.Cu at (82.5, 133.3)
- added P10: DISPLAY_STECKER, toni:micro_match5x2, F.Cu at (118.1, 142.2)
- added P2: DISPLAY_STECKER, toni:micro_match5x2, F.Cu at (167.6, 3.81)
- added P5: IP+, toni:power_terminal, F.Cu at (194.3, 87.6)
- added P6: IP-, toni:power_terminal, F.Cu at (154.9, 87.6)
- added P8: CONN_01X01, Connect:SIL-1, F.Cu at (144.8, 105.4)
- added R17: 10k, SMD_Packages:SMD-0805, F.Cu at (177.8, 114.3)
- added U1: ACS758, toni:ACS758_PFF, F.Cu at (175.3, 106.7)
- added U4: RD-0512D, toni:RD-xx12D, F.Cu at (204.5, 124.5)
- added Y1: RESONATEUR, toni:CerOsc_3,2x1,3, F.Cu at (133.3, 141.0)
- moved R9 5.80 mm to (143.5, 108.0)
- moved R7 4.89 mm to (152.4, 108.0)
- moved R6 4.44 mm to (152.4, 102.9)
- moved R5 3.92 mm to (152.4, 105.4)
- moved R8 2.95 mm to (148.6, 108.0)
- moved D2 2.14 mm to (148.6, 102.9)
- moved C11 1.68 mm to (148.6, 106.7)

Commit message: work
Parts:
- added display_board: EuroBoard_viertel_Type-I_80mmX50mm_holes, EuroBoard_Outline:EuroBoard_viertel_Type-I_80mmX50mm_holes, F.Cu at (178.8, 122.9)
- added main: EuroBoard_halb_Type-I_100mmX80mm_holes, EuroBoard_Outline:EuroBoard_halb_Type-I_100mmX80mm_holes, F.Cu at (67.8, 152.9)
- moved C22 99.3 mm to (152.1, 135.3)
- moved R12 99.3 mm to (142.0, 135.3)
- moved C20 99.3 mm to (148.3, 127.6)
- moved C23 99.3 mm to (144.5, 136.5)
- moved P12 99.3 mm to (158.5, 134.0)
- moved R13 99.3 mm to (143.3, 131.4)
- moved R16 99.3 mm to (148.3, 130.2)
- moved U6 99.3 mm to (148.3, 135.3)
- moved DISP1 92.1 mm to (219.2, 108.2)
- moved P2 87.6 mm to (209.0, 81.0), turned to 90 degrees
- moved U5 80.5 mm to (149.4, 92.3)
- moved C18 80.5 mm to (149.4, 88.5)
- moved C19 80.5 mm to (153.2, 93.6)
- moved C21 80.5 mm to (160.8, 91.1)
- moved R14 80.5 mm to (155.7, 93.6)
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Connections:
- IC1 pad 19: Net-(IC1-Pad19) -> GND
Routing:
- net GND: track 0.00 -> 118.0 mm
- net VCC: track 0.00 -> 100.9 mm
- net AGND: track 0.00 -> 40.3 mm
- net /CSB_D: track 0.00 -> 36.0 mm
- net /RS_D: track 0.00 -> 21.1 mm
- net /B_D: track 0.00 -> 18.1 mm
- net Net-(P6-Pad1): track 0.00 -> 17.2 mm
- net Net-(P5-Pad1): track 0.00 -> 17.2 mm
- net /S_D: track 0.00 -> 13.6 mm
- net Net-(F1-Pad1): track 0.00 -> 13.5 mm
- net /A_D: track 0.00 -> 12.5 mm
- net Net-(P11-Pad2): track 0.00 -> 8.43 mm
- net +5VA: track 0.00 -> 7.99 mm
- net Net-(P11-Pad1): track 0.00 -> 5.89 mm
- net Net-(C4-Pad1): track 0.00 -> 5.53 mm
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Other:
- board outline added: 100 x 80 mm

Commit message: work
Parts:
- added C25: 100nF, SMD_Packages:SMD-0603, F.Cu at (89.9, 104.6)
- added C26: C, SMD_Packages:SMD-0603, F.Cu at (122.2, 106.4)
- P1, P11, P12, P4, P7, SP1, U4: moved to B.Cu
- moved C5 49.7 mm to (93.2, 75.4), turned to 180 degrees
- moved R5 35.0 mm to (96.5, 118.6), turned to 90 degrees
- moved R7 28.5 mm to (91.7, 101.3), turned to 270 degrees
- moved R12 28.1 mm to (162.8, 116.3)
- moved R8 25.9 mm to (91.7, 104.6), turned to 270 degrees
- moved C23 23.4 mm to (159.5, 118.6), turned to 0 degrees
- moved R10 21.1 mm to (125.0, 110.5), turned to 270 degrees
- moved R13 19.9 mm to (162.1, 125.0), turned to 270 degrees
- moved R6 19.2 mm to (105.2, 102.4), turned to 180 degrees
- moved R9 19.0 mm to (125.0, 106.9), turned to 270 degrees
- moved U6 18.0 mm to (159.3, 120.9), turned to 90 degrees
- moved SP1 17.9 mm to (88.6, 121.7)
- moved P8 17.9 mm to (125.0, 104.1)
- moved C11 17.8 mm to (129.3, 104.6)
- moved P3 16.9 mm to (115.6, 109.2)
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Connections:
- P4 pad 2: Net-(IC1-Pad28) -> Net-(IC1-Pad27)
- P4 pad 3: Net-(IC1-Pad27) -> Net-(IC1-Pad28)
- P7 pad 2: Net-(IC1-Pad31) -> Net-(IC1-Pad30)
- P7 pad 3: Net-(IC1-Pad30) -> Net-(IC1-Pad31)
Routing:
- net /MOSI: track 0.00 -> 112.3 mm, vias 0 -> 3
- net VCC: track 100.9 -> 202.1 mm
- net /SCK: track 0.00 -> 96.1 mm, vias 0 -> 4
- net GND: track 118.0 -> 209.8 mm, vias 0 -> 2
- net /SS_DAC: track 3.65 -> 48.7 mm
- net /MISO: track 0.00 -> 40.6 mm, vias 0 -> 2
- net AGND: track 40.3 -> 80.2 mm, vias 0 -> 3
- net /A: track 0.00 -> 36.7 mm
- net /CSB: track 0.00 -> 26.9 mm
- net /U_reserve: track 0.00 -> 26.2 mm, vias 0 -> 2
- net Net-(IC1-Pad28): track 0.00 -> 25.8 mm
- net Net-(P1-Pad3): track 0.00 -> 23.6 mm
- net Net-(IC1-Pad27): track 0.00 -> 23.1 mm
- net /SCK_D: track 0.00 -> 22.6 mm, vias 0 -> 2
- net /S: track 0.00 -> 22.5 mm
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
Commit message: layout fertig
Parts:
- added C27: 100nF, SMD_Packages:SMD-0402, F.Cu at (202.9, 90.4)
- moved C7 50.1 mm to (191.5, 93.2), turned to 0 degrees
- moved C9 17.5 mm to (228.3, 91.2), turned to 180 degrees
- moved C8 11.8 mm to (233.4, 84.8), turned to 270 degrees
- moved C6 11.2 mm to (233.2, 90.2)
- moved R15 9.76 mm to (150.1, 97.8), turned to 0 degrees
- moved C18 8.93 mm to (142.5, 94.2), turned to 270 degrees
- moved C21 7.26 mm to (154.7, 95.0), turned to 270 degrees
- moved R14 5.66 mm to (150.1, 94.5), turned to 180 degrees
- moved C17 4.02 mm to (145.0, 96.0)
- moved C19 3.86 mm to (150.4, 96.3), turned to 180 degrees
- moved U5 1.08 mm to (150.1, 91.6)
Routing:
- net GND: track 209.8 -> 422.1 mm, vias 2 -> 10
- net VCC: track 202.1 -> 365.0 mm, vias 0 -> 8
- net +12V: track 1.69 -> 68.5 mm, vias 0 -> 2
- net AGND: track 80.2 -> 140.0 mm
- net +5VA: track 7.99 -> 48.0 mm, vias 0 -> 3
- net /U_Strom: track 2.72 -> 33.7 mm
- net -12V: track 2.12 -> 33.1 mm, vias 0 -> 2
- net Net-(C19-Pad2): track 0.00 -> 20.5 mm, vias 0 -> 2
- net Net-(C18-Pad1): track 0.00 -> 8.35 mm, vias 0 -> 2
- net /MISO: track 40.6 -> 42.5 mm
- net /U_reserve: track 26.2 -> 24.6 mm
- net Net-(R3-Pad2): track 8.76 -> 9.91 mm
- net /RST: track 17.4 -> 18.0 mm

Commit message: ps files added
Parts:
- added R18: 4,7k, SMD_Packages:SMD-0805, F.Cu at (112.4, 91.6)
- added R19: 4,7k, SMD_Packages:SMD-0805, F.Cu at (121.9, 94.5)
- added R20: 1k, SMD_Packages:SMD-0805, F.Cu at (101.3, 98.4)
- added R21: 1k, SMD_Packages:SMD-0805, F.Cu at (102.0, 92.2)
Connections:
- net Net-(IC1-Pad27) renamed /SDA
- net Net-(IC1-Pad28) renamed /SCL
- P7 pad 2: Net-(IC1-Pad30) -> Net-(P7-Pad2)
- P7 pad 3: Net-(IC1-Pad31) -> Net-(P7-Pad3)
Routing:
- net Net-(IC1-Pad30): track 16.7 -> 6.68 mm
- net Net-(P7-Pad2): track 0.00 -> 8.41 mm
- net GND: track 422.1 -> 429.3 mm, vias 10 -> 11
- net +5VA: track 48.0 -> 54.2 mm, vias 3 -> 4
- net Net-(P7-Pad3): track 0.00 -> 5.75 mm
- net Net-(IC1-Pad31): track 18.8 -> 13.5 mm
- net /SDA: track 23.1 -> 28.3 mm
- net VCC: track 365.0 -> 368.5 mm
- net Net-(D2-Pad1): track 0.00 -> 1.33 mm
- net /SCL: track 25.8 -> 26.5 mm
- added copper zone on B.Cu, net AGND
- added copper zone on B.Cu, net GND
- added copper zone on F.Cu, net GND

Commit message: kleine Änderungen
Parts:
- added U7: LM4040, SMD_Packages:SOT-23, B.Cu at (111.9, 112.9)
Routing:
- net Net-(C4-Pad1): track 5.42 -> 15.3 mm, vias 0 -> 1
- net GND: track 429.3 -> 438.3 mm
- net /SCK: track 95.9 -> 99.6 mm
- net VCC: track 368.5 -> 366.0 mm
- net /RST: track 18.0 -> 18.6 mm
- added copper zone on F.Cu, net VCC
