File: server_lader.sch (KiCad schematic (older format))
At the start: 67 parts, among them IC1 ATMEGA168PA-A, IC2 DAC8560, P1 5V_Vbatt, P10 DISPLAY_STECKER, P11 on/off, P12 A_regulation_out, P2 DISPLAY_STECKER, P3 CONN_02X03, P4 I2C, P5 IP+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

Commit message: work
Parts:
- removed X1: Resonator CSTCE16M0V53, symbol CRYSTAL_SMD
- added Y1: RESONATEUR, toni:CerOsc_3,2x1,3, symbol RESONATEUR
- C24: renamed from C?; footprint (none) -> SMD_Packages:SMD-0603
- D1: footprint (none) -> Diodes_SMD:Diode-Universal-SMA-SMB_Handsoldering
- P10, P2: footprint (none) -> toni:micro_match5x2
- P5, P6: footprint (none) -> toni:power_terminal
- P8: footprint (none) -> Connect:SIL-1
- R17: renamed from R?; footprint (none) -> SMD_Packages:SMD-0805
- U1: footprint (none) -> toni:ACS758_PFF
- U4: footprint (none) -> toni:RD-xx12D
Connections:
- net GND: now also Y1.2
- net at IC1.7 ((PCINT6/XTAL1/TOSC1)PB6): now also Y1.3
- net at IC1.8 ((PCINT7/XTAL2/TOSC2)PB7): now also Y1.1
Changed lines of the file:
@@
 EESchema Schematic File Version 2
-LIBS:toni
 LIBS:power
 LIBS:device
@@
 LIBS:contrib
 LIBS:valves
-LIBS:dac8560
+LIBS:toni
 LIBS:server_lader-cache
 EELAYER 25 0
@@
 F 0 "D1" H 1650 1050 50  0000 C CNN
 F 1 "ZENER 5,6V" H 1650 850 40  0000 C CNN
-F 2 "" H 1650 950 60  0001 C CNN
+F 2 "Diodes_SMD:Diode-Universal-SMA-SMB_Handsoldering" H 1650 950 60  0001 C CNN
 F 3 "" H 1650 950 60  0000 C CNN
 	1    1650 950
@@
 F 0 "P10" H 5900 2050 50  0000 C CNN
 F 1 "DISPLAY_STECKER" H 5900 1450 50  0000 C CNN
-F 2 "" H 5900 550 60  0001 C CNN
+F 2 "toni:micro_match5x2" H 5900 550 60  0001 C CNN
 F 3 "" H 5900 550 60  0000 C CNN
 	1    5900 1750
@@
 F 0 "U4" H 7150 1450 60  0000 C CNN
 F 1 "RD-0512D" H 7150 1900 60  0000 C CNN
-F 2 "" H 7750 1650 60  0001 C CNN
+F 2 "toni:RD-xx12D" H 7750 1650 60  0001 C CNN
 F 3 "" H 7750 1650 60  0000 C CNN
 	1    7150 1650
@@
 F 0 "P8" H 5200 800 50  0000 C CNN
 F 1 "CONN_01X01" V 5300 700 50  0000 C CNN
-F 2 "" H 5200 700 60  0001 C CNN
+F 2 "Connect:SIL-1" H 5200 700 60  0001 C CNN
 F 3 "" H 5200 700 60  0000 C CNN
 	1    5200 700
@@
 F 0 "P5" H 4550 4100 50  0000 C CNN
 F 1 "IP+" V 4650 4000 50  0000 C CNN
-F 2 "" H 4550 4000 60  0001 C CNN
+F 2 "toni:power_terminal" H 4550 4000 60  0001 C CNN
 F 3 "" H 4550 4000 60  0000 C CNN
 	1    4550 4000
@@
 F 0 "P6" H 4550 4800 50  0000 C CNN
 F 1 "IP-" V 4650 4700 50  0000 C CNN
-F 2 "" H 4550 4700 60  0001 C CNN
+F 2 "toni:power_terminal" H 4550 4700 60  0001 C CNN
 F 3 "" H 4550 4700 60  0000 C CNN
 	1    4550 4700
@@
 F 0 "U1" H 5500 4000 60  0000 C CNN
 F 1 "ACS758" H 5100 4650 60  0000 C CNN
-F 2 "" H 4950 4350 60  0001 C CNN
+F 2 "toni:ACS758_PFF" H 4950 4350 60  0001 C CNN
 F 3 "" H 4950 4350 60  0000 C CNN
 	1    4950 4350
@@
 F 0 "P2" H 1100 7500 50  0000 C CNN
 F 1 "DISPLAY_STECKER" H 1100 6900 50  0000 C CNN
-F 2 "" H 1100 6000 60  0001 C CNN
+F 2 "toni:micro_match5x2" H 1100 6000 60  0001 C CNN
 F 3 "" H 1100 6000 60  0000 C CNN
 	1    1100 7200
@@
 	1    0    0    -1
 $EndComp
-$Comp
-L CRYSTAL_SMD X1
-U 1 1 54650B0C
-P 2900 1000
-F 0 "X1" H 3100 900 60  0000 C CNN
-F 1 "Resonator CSTCE16M0V53" H 2900 1200 60  0000 C CNN
-F 2 "" H 2900 1000 60  0001 C CNN
-F 3 "" H 2900 1000 60  0000 C CNN
-	1    2900 1000
-	1    0    0    -1
-$EndComp
 Wire Wire Line
 	3200 1000 4350 1000
@@
 L GND #PWR094
 U 1 1 54651961
-P 2900 1250
-F 0 "#PWR094" H 2900 1250 30  0001 C CNN
-F 1 "GND" H 2900 1180 30  0001 C CNN
-F 2 "" H 2900 1250 60  0000 C CNN
-F 3 "" H 2900 1250 60  0000 C CNN
-	1    2900 1250
+P 2900 1300
+F 0 "#PWR094" H 2900 1300 30  0001 C CNN
+F 1 "GND" H 2900 1230 30  0001 C CNN
+F 2 "" H 2900 1300 60  0000 C CNN
+F 3 "" H 2900 1300 60  0000 C CNN
+	1    2900 1300
 	1    0    0    -1
 $EndComp
@@
 	3900 2650 3900 2550
 $Comp
-L R R?
+L R R17
 U 1 1 546588C7
 P 5900 4500
-F 0 "R?" V 5980 4500 40  0000 C CNN
+F 0 "R17" V 5980 4500 40  0000 C CNN
 F 1 "10k" V 5907 4501 40  0000 C CNN
-F 2 "" V 5830 4500 30  0000 C CNN
+F 2 "SMD_Packages:SMD-0805" V 5830 4500 30  0001 C CNN
 F 3 "" H 5900 4500 30  0000 C CNN
 	1    5900 4500
@@
 $EndComp
 $Comp
-L C C?
+L C C24
 U 1 1 5465917C
 P 6150 4700
-F 0 "C?" H 6150 4800 40  0000 L CNN
+F 0 "C24" H 6150 4800 40  0000 L CNN
 F 1 "1uF" H 6156 4615 40  0000 L CNN
-F 2 "" H 6188 4550 30  0000 C CNN
+F 2 "SMD_Packages:SMD-0603" H 6188 4550 30  0001 C CNN
 F 3 "" H 6150 4700 60  0000 C CNN
 	1    6150 4700
@@
 $EndComp
 $Comp
-L GND #PWR?
+L GND #PWR0102
 U 1 1 546591E2
 P 6150 4900
-F 0 "#PWR?" H 6150 4900 30  0001 C CNN
+F 0 "#PWR0102" H 6150 4900 30  0001 C CNN
 F 1 "GND" H 6150 4830 30  0001 C CNN
 F 2 "" H 6150 4900 60  0000 C CNN
@@
 	1    0    0    -1
 $EndComp
+$Comp
+L RESONATEUR Y1
+U 1 1 54667D59
+P 2900 1050
+F 0 "Y1" H 2920 1250 60  0000 C CNN
+F 1 "RESONATEUR" H 3330 850 60  0000 C CNN
+F 2 "toni:CerOsc_3,2x1,3" H 2900 1050 60  0001 C CNN
+F 3 "" H 2900 1050 60  0000 C CNN
+	1    2900 1050
+	1    0    0    -1
+$EndComp

Commit message: work
Connections:
- net GND: now also IC1.19 (ADC6)
- no-connect marks 8 -> 7
Changed lines of the file:
@@
 $EndComp
 NoConn ~ 3700 1600
-NoConn ~ 1800 2850
 NoConn ~ 1800 2950
 $Comp
@@
 	1    0    0    -1
 $EndComp
+$Comp
+L GND #PWR?
+U 1 1 5466ABD3
+P 1800 2850
+F 0 "#PWR?" H 1800 2850 30  0001 C CNN
+F 1 "GND" H 1800 2780 30  0001 C CNN
+F 2 "" H 1800 2850 60  0000 C CNN
+F 3 "" H 1800 2850 60  0000 C CNN
+	1    1800 2850
+	0    1    1    0
+$EndComp
 $EndSCHEMATC

Commit message: work
Parts:
- added C25: 100nF, SMD_Packages:SMD-0603, symbol C
- added C26: C, SMD_Packages:SMD-0603, symbol C
Connections:
- net GND: now also C25.2, C26.2
- net U_Netzteil: now also C25.1
- net U_reserve: now also C26.1
- net at IC1.27 ((PCINT12/SDA/ADC4)PC4): now also P4.2 (P2); no longer P4.3 (P3)
- net at IC1.28 ((PCINT14/SCL/ADC5)PC5): now also P4.3 (P3); no longer P4.2 (P2)
- net at IC1.30 ((PCINT16/RXD)PD0): now also P7.2 (P2); no longer P7.3 (P3)
- net at IC1.31 ((PCINT17/TXD)PD1): now also P7.3 (P3); no longer P7.2 (P2)
Changed lines of the file:
@@
 	3700 1800 4000 1800
 Wire Wire Line
-	3700 3200 4150 3200
-Wire Wire Line
-	4150 3200 4150 3100
-Wire Wire Line
-	4150 3100 4450 3100
-Wire Wire Line
-	3700 3100 4050 3100
-Wire Wire Line
-	4050 3100 4050 3150
-Wire Wire Line
-	4050 3150 4250 3150
-Wire Wire Line
-	4250 3150 4250 3200
-Wire Wire Line
-	4250 3200 4450 3200
+	3700 3100 4450 3100
 Wire Wire Line
 	1350 750  1950 750
@@
 	0    1    1    0
 $EndComp
-Wire Wire Line
-	3700 2750 4050 2750
-Wire Wire Line
-	3700 2850 4050 2850
 $Comp
 L PWR_FLAG #FLG090
@@
 $EndComp
 $Comp
-L GND #PWR?
+L GND #PWR0103
 U 1 1 5466ABD3
 P 1800 2850
-F 0 "#PWR?" H 1800 2850 30  0001 C CNN
+F 0 "#PWR0103" H 1800 2850 30  0001 C CNN
 F 1 "GND" H 1800 2780 30  0001 C CNN
 F 2 "" H 1800 2850 60  0000 C CNN
@@
 	0    1    1    0
 $EndComp
+Wire Wire Line
+	3700 3200 4450 3200
+Wire Wire Line
+	3700 2850 3900 2850
+Wire Wire Line
+	3900 2850 3900 2750
+Wire Wire Line
+	3900 2750 4050 2750
+Wire Wire Line
+	3700 2750 3700 2800
+Wire Wire Line
+	3700 2800 4050 2800
+Wire Wire Line
+	4050 2800 4050 2850
+$Comp
+L C C25
+U 1 1 5466D39F
+P 4900 1650
+F 0 "C25" H 4900 1750 40  0000 L CNN
+F 1 "100nF" H 4906 1565 40  0000 L CNN
+F 2 "SMD_Packages:SMD-0603" H 4938 1500 30  0001 C CNN
+F 3 "" H 4900 1650 60  0000 C CNN
+	1    4900 1650
+	1    0    0    -1
+$EndComp
+Wire Wire Line
+	4700 1400 4900 1400
+Wire Wire Line
+	4900 1400 4900 1450
+Wire Wire Line
+	4700 1900 4900 1900
+Wire Wire Line
+	4900 1900 4900 1850
+$Comp
+L C C26
+U 1 1 5466D714
+P 5400 1650
+F 0 "C26" H 5400 1750 40  0000 L CNN
+F 1 "C" H 5406 1565 40  0000 L CNN
+F 2 "SMD_Packages:SMD-0603" H 5438 1500 30  0001 C CNN
+F 3 "" H 5400 1650 60  0000 C CNN
+	1    5400 1650
+	1    0    0    -1
+$EndComp
+Wire Wire Line
+	5200 1400 5400 1400
+Wire Wire Line
+	5400 1400 5400 1450
+Wire Wire Line
+	5200 1900 5400 1900
+Wire Wire Line
+	5400 1900 5400 1850
 $EndSCHEMATC

Commit message: layout fertig
Parts:
- added C27: 100nF, SMD_Packages:SMD-0402, symbol C
Connections:
- net GND: now also C27.2
- net VCC: now also C27.1
Changed lines of the file:
@@
 Wire Wire Line
 	5400 1900 5400 1850
+$Comp
+L GND #PWR0104
+U 1 1 5467C6CE
+P 5150 6450
+F 0 "#PWR0104" H 5150 6450 30  0001 C CNN
+F 1 "GND" H 5150 6380 30  0001 C CNN
+F 2 "" H 5150 6450 60  0000 C CNN
+F 3 "" H 5150 6450 60  0000 C CNN
+	1    5150 6450
+	1    0    0    -1
+$EndComp
+$Comp
+L C C27
+U 1 1 5467C6D4
+P 5150 6250
+F 0 "C27" H 5150 6350 40  0000 L CNN
+F 1 "100nF" H 5156 6165 40  0000 L CNN
+F 2 "SMD_Packages:SMD-0402" H 5188 6100 30  0001 C CNN
+F 3 "" H 5150 6250 60  0000 C CNN
+	1    5150 6250
+	1    0    0    -1
+$EndComp
+$Comp
+L VCC #PWR0105
+U 1 1 5467C6DA
+P 5150 6050
+F 0 "#PWR0105" H 5150 6150 30  0001 C CNN
+F 1 "VCC" H 5150 6150 30  0000 C CNN
+F 2 "" H 5150 6050 60  0000 C CNN
+F 3 "" H 5150 6050 60  0000 C CNN
+	1    5150 6050
+	1    0    0    -1
+$EndComp
 $EndSCHEMATC

Commit message: ps files added
Parts:
- added R18, R19: 4,7k, SMD_Packages:SMD-0805, symbol R
- added R20, R21: 1k, SMD_Packages:SMD-0805, symbol R
Connections:
- net VCC: now also R18.1, R19.1
- net SDA: now reaches IC1.27 ((PCINT12/SDA/ADC4)PC4), P4.2 (P2)
- net SDA: now also R19.2
- net SCL: now reaches IC1.28 ((PCINT14/SCL/ADC5)PC5), P4.3 (P3)
- net SCL: now also R18.2
- net at IC1.30 ((PCINT16/RXD)PD0): now also R20.2; no longer P7.2 (P2)
- net at IC1.31 ((PCINT17/TXD)PD1): now also R21.2; no longer P7.3 (P3)
- new net: P7.2 (P2), R20.1
- new net: P7.3 (P3), R21.1
Changed lines of the file:
@@
 	3700 1800 4000 1800
-Wire Wire Line
-	3700 3100 4450 3100
 Wire Wire Line
 	1350 750  1950 750
@@
 $EndComp
 Wire Wire Line
-	3700 3200 4450 3200
-Wire Wire Line
 	3700 2850 3900 2850
 Wire Wire Line
@@
 	1    0    0    -1
 $EndComp
+$Comp
+L R R20
+U 1 1 5467BC23
+P 4050 3100
+F 0 "R20" V 4130 3100 40  0000 C CNN
+F 1 "1k" V 4057 3101 40  0000 C CNN
+F 2 "SMD_Packages:SMD-0805" V 3980 3100 30  0001 C CNN
+F 3 "" H 4050 3100 30  0000 C CNN
+	1    4050 3100
+	0    1    1    0
+$EndComp
+$Comp
+L R R21
+U 1 1 5467BCF3
+P 4050 3200
+F 0 "R21" V 4130 3200 40  0000 C CNN
+F 1 "1k" V 4057 3201 40  0000 C CNN
+F 2 "SMD_Packages:SMD-0805" V 3980 3200 30  0001 C CNN
+F 3 "" H 4050 3200 30  0000 C CNN
+	1    4050 3200
+	0    1    1    0
+$EndComp
+Wire Wire Line
+	4300 3100 4450 3100
+Wire Wire Line
+	3700 3100 3800 3100
+Wire Wire Line
+	3700 3200 3800 3200
+Wire Wire Line
+	4300 3200 4450 3200
+Text Label 3700 2750 0    60   ~ 0
+SDA
+Text Label 3700 2850 0    60   ~ 0
+SCL
+Text Label 1300 4350 0    60   ~ 0
+SDA
+Text Label 950  4350 0    60   ~ 0
+SCL
+$Comp
+L R R18
+U 1 1 5467CCF6
+P 950 4100
+F 0 "R18" V 1030 4100 40  0000 C CNN
+F 1 "4,7k" V 957 4101 40  0000 C CNN
+F 2 "SMD_Packages:SMD-0805" V 880 4100 30  0001 C CNN
+F 3 "" H 950 4100 30  0000 C CNN
+	1    950  4100
+	1    0    0    -1
+$EndComp
+$Comp
+L R R19
+U 1 1 5467CE54
+P 1300 4100
+F 0 "R19" V 1380 4100 40  0000 C CNN
+F 1 "4,7k" V 1307 4101 40  0000 C CNN
+F 2 "SMD_Packages:SMD-0805" V 1230 4100 30  0001 C CNN
+F 3 "" H 1300 4100 30  0000 C CNN
+	1    1300 4100
+	1    0    0    -1
+$EndComp
+$Comp
+L VCC #PWR0106
+U 1 1 5467CF50
+P 950 3850
+F 0 "#PWR0106" H 950 3950 30  0001 C CNN
+F 1 "VCC" H 950 3950 30  0000 C CNN
+F 2 "" H 950 3850 60  0000 C CNN
+F 3 "" H 950 3850 60  0000 C CNN
+	1    950  3850
+	1    0    0    -1
+$EndComp
+$Comp
+L VCC #PWR0107
+U 1 1 5467CFA5
+P 1300 3850
+F 0 "#PWR0107" H 1300 3950 30  0001 C CNN
+F 1 "VCC" H 1300 3950 30  0000 C CNN
+F 2 "" H 1300 3850 60  0000 C CNN
+F 3 "" H 1300 3850 60  0000 C CNN
+	1    1300 3850
+	1    0    0    -1
+$EndComp

Commit message: kleine Änderungen
Parts:
- added U7: LM4040, SMD_Packages:SOT-23, symbol LM4040
Connections:
- net GND: now also U7.2 (GND)
- net at C4.1, IC1.20 (AREF), R1.2: now also U7.1 (V+)

Commit message: bugfixes
Parts:
- C4: value 100uF -> 100nF
- R7: value 12k -> 15k
Changed lines of the file:
@@
 P 1200 2300
 F 0 "C4" H 1200 2400 40  0000 L CNN
-F 1 "100uF" H 1206 2215 40  0000 L CNN
+F 1 "100nF" H 1206 2215 40  0000 L CNN
 F 2 "SMD_Packages:SMD-0402" H 1238 2150 30  0001 C CNN
 F 3 "" H 1200 2300 60  0000 C CNN
@@
 P 4700 1150
 F 0 "R7" V 4780 1150 40  0000 C CNN
-F 1 "12k" V 4707 1151 40  0000 C CNN
+F 1 "15k" V 4707 1151 40  0000 C CNN
 F 2 "SMD_Packages:SMD-0805" V 4630 1150 30  0001 C CNN
 F 3 "" H 4700 1150 30  0000 C CNN

Commit message: neue Dateien - Version so gefertigt.
Parts:
- R14: value R1 -> 33k
- R15: value R2 -> 10k
Other:
- note added: "RFB = 10k\nRG1 = 3,3k\nRG2 = 10k"
Changed lines of the file:
@@
 LIBS:contrib
 LIBS:valves
-LIBS:toni
 LIBS:server_lader-cache
 EELAYER 25 0
@@
 P 10350 1700
 F 0 "R14" V 10430 1700 40  0000 C CNN
-F 1 "R1" V 10357 1701 40  0000 C CNN
+F 1 "33k" V 10357 1701 40  0000 C CNN
 F 2 "SMD_Packages:SMD-0805" V 10280 1700 30  0001 C CNN
 F 3 "" H 10350 1700 30  0000 C CNN
@@
 P 10350 2200
 F 0 "R15" V 10430 2200 40  0000 C CNN
-F 1 "R2" V 10357 2201 40  0000 C CNN
+F 1 "10k" V 10357 2201 40  0000 C CNN
 F 2 "SMD_Packages:SMD-0805" V 10280 2200 30  0001 C CNN
 F 3 "" H 10350 2200 30  0000 C CNN
@@
 	1    0    0    -1
 $EndComp
+Text Notes 9200 4400 0    60   ~ 0
+RFB = 10k\nRG1 = 3,3k\nRG2 = 10k
 $EndSCHEMATC
